File: Hardware/XBee-Explorer-Dongle.brd (EAGLE design)
At the start: 40.6 x 27.9 mm, 37 parts, among them U2 XBEE-1B3, U3 MIC5219 3.3V, U4 FTS31XS-U

Commit message: Changed font to Vector, and re arranged SPK logo
Parts:
- moved LOGO2 1.45 mm to (34.4, 11.0)
Changed lines of the file:
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@@
 <?xml version="1.0" encoding="utf-8"?>
 <!DOCTYPE eagle SYSTEM "eagle.dtd">
-<eagle version="6.4">
+<eagle version="7.1.0">
 <drawing>
 <settings>
@@
 <layer number="47" name="Measures" color="7" fill="1" visible="no" active="yes"/>
 <layer number="48" name="Document" color="7" fill="1" visible="no" active="yes"/>
-<layer number="49" name="Reference" color="7" fill="1" visible="no" active="yes"/>
+<layer number="49" name="Reference" color="7" fill="1" visible="yes" active="yes"/>
 <layer number="50" name="dxf" color="7" fill="1" visible="no" active="yes"/>
 <layer number="51" name="tDocu" color="6" fill="1" visible="yes" active="yes"/>
@@
 <wire x1="0" y1="0" x2="40.64" y2="0" width="0.2032" layer="20"/>
 <text x="9.017" y="17.78" size="1.016" layer="21" ratio="15" align="center">PWR</text>
-<text x="37.338" y="9.525" size="1.016" layer="21" ratio="15" align="center-right">TX</text>
-<text x="37.338" y="8.255" size="1.016" layer="21" ratio="15" align="center-right">RX</text>
-<text x="37.338" y="19.685" size="1.016" layer="21" ratio="15" align="center-right">RSSI</text>
-<text x="33.528" y="20.066" size="1.016" layer="22" ratio="15" rot="MR270">3.3V</text>
-<text x="30.988" y="20.066" size="1.016" layer="22" ratio="15" rot="MR270">DOUT</text>
-<text x="28.448" y="20.066" size="1.016" layer="22" ratio="15" rot="MR270">DIN</text>
-<text x="25.908" y="20.066" size="1.016" layer="22" ratio="15" rot="MR270">DIO12</text>
-<text x="23.368" y="20.066" size="1.016" layer="22" ratio="15" rot="MR270">RST</text>
-<text x="20.828" y="20.066" size="1.016" layer="22" ratio="15" rot="MR270">RSSI</text>
-<text x="18.288" y="20.066" size="1.016" layer="22" ratio="15" rot="MR270">DIO11</text>
-<text x="15.748" y="20.066" size="1.016" layer="22" ratio="15" rot="MR270">RES</text>
-<text x="13.208" y="20.066" size="1.016" layer="22" ratio="15" rot="MR270">DTR</text>
-<text x="10.668" y="20.066" size="1.016" layer="22" ratio="15" rot="MR270">GND</text>
-<text x="35.052" y="7.874" size="1.016" layer="22" ratio="15" rot="MR90">DIO0</text>
-<text x="32.512" y="7.874" size="1.016" layer="22" ratio="15" rot="MR90">DIO1</text>
-<text x="29.972" y="7.874" size="1.016" layer="22" ratio="15" rot="MR90">DIO2</text>
-<text x="27.432" y="7.874" size="1.016" layer="22" ratio="15" rot="MR90">DIO3</text>
-<text x="24.892" y="7.874" size="1.016" layer="22" ratio="15" rot="MR90">RTS</text>
-<text x="22.352" y="7.874" size="1.016" layer="22" ratio="15" rot="MR90">DIO5</text>
-<text x="19.812" y="7.874" size="1.016" layer="22" ratio="15" rot="MR90">RES</text>
-<text x="17.272" y="7.874" size="1.016" layer="22" ratio="15" rot="MR90">DIO9</text>
-<text x="14.732" y="7.874" size="1.016" layer="22" ratio="15" rot="MR90">CTS</text>
-<text x="12.192" y="7.874" size="1.016" layer="22" ratio="15" rot="MR90">DIO4</text>
+<text x="37.338" y="9.525" size="1.016" layer="21" font="vector" ratio="15" align="center-right">TX</text>
+<text x="37.338" y="8.255" size="1.016" layer="21" font="vector" ratio="15" align="center-right">RX</text>
+<text x="37.338" y="19.685" size="1.016" layer="21" font="vector" ratio="15" align="center-right">RSSI</text>
+<text x="33.528" y="20.066" size="0.889" layer="22" font="vector" ratio="15" rot="MR270">3.3V</text>
+<text x="30.988" y="20.066" size="0.889" layer="22" font="vector" ratio="15" rot="MR270">DOUT</text>
+<text x="28.448" y="20.066" size="0.889" layer="22" font="vector" ratio="15" rot="MR270">DIN</text>
+<text x="25.908" y="20.066" size="0.889" layer="22" font="vector" ratio="15" rot="MR270">DIO12</text>
+<text x="23.368" y="20.066" size="0.889" layer="22" font="vector" ratio="15" rot="MR270">RST</text>
+<text x="20.828" y="20.066" size="0.889" layer="22" font="vector" ratio="15" rot="MR270">RSSI</text>
+<text x="18.288" y="20.066" size="0.889" layer="22" font="vector" ratio="15" rot="MR270">DIO11</text>
+<text x="15.748" y="20.066" size="0.889" layer="22" font="vector" ratio="15" rot="MR270">RES</text>
+<text x="13.208" y="20.066" size="0.889" layer="22" font="vector" ratio="15" rot="MR270">DTR</text>
+<text x="10.668" y="20.066" size="0.889" layer="22" font="vector" ratio="15" rot="MR270">GND</text>
+<text x="35.052" y="7.874" size="0.889" layer="22" font="vector" ratio="15" rot="MR90">DIO0</text>
+<text x="32.512" y="7.874" size="0.889" layer="22" font="vector" ratio="15" rot="MR90">DIO1</text>
+<text x="29.972" y="7.874" size="0.889" layer="22" font="vector" ratio="15" rot="MR90">DIO2</text>
+<text x="27.432" y="7.874" size="0.889" layer="22" font="vector" ratio="15" rot="MR90">DIO3</text>
+<text x="24.892" y="7.874" size="0.889" layer="22" font="vector" ratio="15" rot="MR90">RTS</text>
+<text x="22.352" y="7.874" size="0.889" layer="22" font="vector" ratio="15" rot="MR90">DIO5</text>
+<text x="19.812" y="7.874" size="0.889" layer="22" font="vector" ratio="15" rot="MR90">RES</text>
+<text x="17.272" y="7.874" size="0.889" layer="22" font="vector" ratio="15" rot="MR90">DIO9</text>
+<text x="14.732" y="7.874" size="0.889" layer="22" font="vector" ratio="15" rot="MR90">CTS</text>
+<text x="12.192" y="7.874" size="0.889" layer="22" font="vector" ratio="15" rot="MR90">DIO4</text>
 <text x="15.367" y="24.384" size="0.4064" layer="27">XBee Socket Up</text>
 <text x="15.621" y="2.413" size="0.4064" layer="27">XBee Socket Up</text>
 <text x="16.256" y="4.445" size="1.27" layer="27">DNP</text>
 <text x="16.256" y="19.812" size="1.27" layer="27">DNP</text>
-<text x="34.925" y="24.638" size="1.016" layer="21" ratio="15">1</text>
-<text x="34.29" y="2.032" size="1.016" layer="21" ratio="15">20</text>
-<text x="9.652" y="7.874" size="1.016" layer="22" ratio="15" rot="MR90">5V</text>
-<text x="36.068" y="20.066" size="1.016" layer="22" ratio="15" rot="MR270">GND</text>
+<text x="34.925" y="24.638" size="1.016" layer="21" font="vector" ratio="15">1</text>
+<text x="34.29" y="2.032" size="1.016" layer="21" font="vector" ratio="15">20</text>
+<text x="9.652" y="7.874" size="0.889" layer="22" font="vector" ratio="15" rot="MR90">5V</text>
+<text x="36.068" y="20.066" size="0.889" layer="22" font="vector" ratio="15" rot="MR270">GND</text>
 <text x="9.398" y="0.381" size="1.4224" layer="16" font="vector" ratio="20" rot="MR0">v23</text>
 <text x="20.32" y="25.781" size="0.889" layer="22" font="vector" ratio="15" rot="MR0" align="center">RSSI</text>
 <wire x1="19.812" y1="24.13" x2="20.828" y2="24.13" width="0.4064" layer="30"/>
 <text x="20.32" y="-10.16" size="1.778" layer="51">Nathan Seidle, Jim Lindblom</text>
-<text x="37.973" y="17.399" size="1.016" layer="21" ratio="15" align="bottom-center">Reset</text>
+<text x="37.973" y="17.399" size="1.016" layer="21" font="vector" ratio="15" align="bottom-center">Reset</text>
 <text x="13.97" y="25.781" size="0.889" layer="22" font="vector" ratio="15" rot="MR0" align="center">DTR</text>
 <text x="16.51" y="2.159" size="0.889" layer="22" font="vector" ratio="15" rot="MR0" align="center">CTS</text>
@@
 <wire x1="23.622" y1="3.81" x2="24.638" y2="3.81" width="0.4064" layer="30"/>
 <text x="2.794" y="-13.081" size="1.778" layer="51">Revised by: Patrick Alberts</text>
-<text x="17.78" y="11.43" size="1.016" layer="22" font="vector" ratio="10" rot="MR180">Xbee Dongle</text>
+<text x="18.669" y="12.192" size="1.016" layer="22" font="vector" ratio="10" rot="MR180">Xbee Dongle</text>
 <dimension x1="45.72" y1="0" x2="45.72" y2="27.94" x3="48.26" y3="13.97" textsize="1.016" textratio="10" layer="47"/>
 <dimension x1="0" y1="36.83" x2="40.64" y2="36.83" x3="20.32" y3="39.37" textsize="1.016" textratio="10" layer="47"/>
@@
 <pass name="Default">
 <param name="RoutingGrid" value="50mil"/>
+<param name="AutoGrid" value="1"/>
+<param name="Efforts" value="0"/>
+<param name="TopRouterVariant" value="1"/>
 <param name="tpViaShape" value="round"/>
 <param name="PrefDir.1" value="|"/>
@@
 </element>
 <element name="LOGO1" library="SparkFun-Aesthetics" package="SFE_LOGO_FLAME_.1" value="SFE_LOGO_FLAME.1_INCH" x="7.62" y="1.27"/>
-<element name="LOGO2" library="SparkFun-Aesthetics" package="SFE_LOGO_NAME_.2" value="SFE_LOGO_NAME.2_INCH" x="33.02" y="11.43" rot="MR0"/>
+<element name="LOGO2" library="SparkFun-Aesthetics" package="SFE_LOGO_NAME_.2" value="SFE_LOGO_NAME.2_INCH" x="34.417" y="11.049" rot="MR0"/>
 </elements>
 <signals>
