File: Hardware/XBee-Explorer-Dongle.sch (EAGLE design)
At the start: 37 parts, among them U2 XBEE-1B3, U3 MIC5219 3.3V, U4 FT231XS

Commit message: Upd to usb pth, 0603, sch changes
Parts:
- removed JP1: USBA-SMD-MALE-LOCKING, SparkFun-Connectors:USBA-SMD-MALE-LOCKING
- removed U$1: LOGO-SFESK, SparkFun:LOGO-SFESK
- removed U$4: LOGO-SFENEW, SparkFun:LOGO-SFENEW
- added JP4: USB-A-H, SparkFun-Connectors:USB-A-H
- added LOGO1: SFE_LOGO_FLAME.1_INCH, SparkFun-Aesthetics:SFE_LOGO_FLAME.1_INCH
- added LOGO2: SFE_LOGO_NAME.2_INCH, SparkFun-Aesthetics:SFE_LOGO_NAME.2_INCH
- C1: device SparkFun:CAP_POL1206 -> SparkFun-Capacitors:10UF-16V-10%(TANT)
- C2: device SparkFun:CAP0603-CAP -> SparkFun-Capacitors:0.1UF-25V(+80/-20%)(0603)
- C3, C4: device SparkFun:CAP0603-CAP -> SparkFun-Capacitors:47PF-50V-5%(0603)
- R1, R11, R3: device SparkFun:RESISTOR0603-RES -> SparkFun-Resistors:1KOHM-1/10W-1%(0603)
- R2, R5: device SparkFun:RESISTOR0603-RES -> SparkFun-Resistors:27OHM1/10W1%(0603)0603-RES
- R4: device SparkFun:RESISTOR0603-RES -> SparkFun-Resistors:330OHM1/10W1%(0603)
- U3: device SparkFun:V_REG_LDOSMD -> SparkFun-PowerIC:V_REG_MIC52193.3V
- U4: value FT231XS -> FTS31XS-U
Connections:
- net 5V: now also JP4.VBUS; no longer JP1.VBUS
- net GND: now also JP4.GND; no longer JP1.GND
- net N$3: now also JP4.D-; no longer JP1.D-
- net N$6: now also JP4.D+; no longer JP1.D+
Other:
- note added: "Revised by: Patrick Alberts"
- note added: "v23"
- note removed: "v22"
- moved on the sheet: JP2, JP3, R11, R4, S2, SJ1, U2

Commit message: QC checklist items complete.
Parts:
- C11, C14: device SparkFun:CAP0603-CAP -> SparkFun-Capacitors:0.1UF-25V(+80/-20%)(0603)
- D1: value RED -> GREEN; device SparkFun-LED:LED-RED0603 -> SparkFun-LED:LED-GREEN0603
- D2: value GREEN -> Yellow; device SparkFun-LED:LED-GREEN0603 -> SparkFun-LED:LED-YELLOW0603
Changed lines of the file:
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@@
 </classes>
 <parts>
-<part name="C11" library="SparkFun" deviceset="CAP" device="0603-CAP" value="0.1uF"/>
+<part name="C11" library="SparkFun-Capacitors" deviceset="0.1UF-25V(+80/-20%)(0603)" device="" value="0.1uF"/>
 <part name="GND20" library="SparkFun" deviceset="GND" device=""/>
 <part name="GND21" library="SparkFun" deviceset="GND" device=""/>
 <part name="R11" library="SparkFun-Resistors" deviceset="1KOHM-1/10W-1%(0603)" device="" value="1K"/>
-<part name="C14" library="SparkFun" deviceset="CAP" device="0603-CAP" value="0.1uF"/>
+<part name="C14" library="SparkFun-Capacitors" deviceset="0.1UF-25V(+80/-20%)(0603)" device="" value="0.1uF"/>
 <part name="GND27" library="SparkFun" deviceset="GND" device=""/>
 <part name="GND28" library="SparkFun" deviceset="GND" device=""/>
@@
 <part name="SJ3" library="SparkFun-Passives" deviceset="SOLDERJUMPER" device="TRACE" value="RSSI"/>
 <part name="SJ4" library="SparkFun-Passives" deviceset="SOLDERJUMPER" device="TRACE" value="RSSI"/>
-<part name="D1" library="SparkFun-LED" deviceset="LED-RED" device="0603" value="RED"/>
-<part name="D2" library="SparkFun-LED" deviceset="LED-GREEN" device="0603" value="GREEN"/>
+<part name="D1" library="SparkFun-LED" deviceset="LED-GREEN" device="0603" value="GREEN"/>
+<part name="D2" library="SparkFun-LED" deviceset="LED-YELLOW" device="0603" value="Yellow"/>
 <part name="D3" library="SparkFun-LED" deviceset="LED-GREEN" device="0603" value="GREEN"/>
 <part name="D4" library="SparkFun-LED" deviceset="LED-RED" device="0603" value="RED"/>
